File: kp_artnet2dmx6.kicad_pcb (KiCad board)
At the start: 2 copper layers, 27 parts, among them IC1 KSZ8081MNXIA-TR, IC2 M95640-RMN6P, IC3 AP2281-3WG-7, IC4 MP2331HGTL-P, J1 RJ45_Amphenol_RJMG1BD3B8K1ANR, J14 SWD, J2 SCREEN, Q1 AO3401A, SW1 SW_SPDT, U1 STM32F407VETx, U2 MCP23S17_SP, U3 USBLC6-2SC6, Y1 ASDDV-25.000MHZ-LC-T

Commit message: all footprints assigned
Parts:
- added C1: 100n, Capacitor_SMD:C_0402_1005Metric, F.Cu at (78.2, 33.1)
- added C10: 100n, Capacitor_SMD:C_0402_1005Metric, F.Cu at (63.7, 32.5)
- added C11: 10n, Capacitor_SMD:C_0402_1005Metric, F.Cu at (25.8, 72.6)
- added C12: 2.2u, Capacitor_SMD:C_0805_2012Metric, F.Cu at (221.6, 59.0)
- added C13: 100n, Capacitor_SMD:C_0402_1005Metric, F.Cu at (225.1, 59.0)
- added C14: 10u, Capacitor_SMD:C_1206_3216Metric, F.Cu at (266.9, 54.0)
- added C15: 100n, Capacitor_SMD:C_0402_1005Metric, F.Cu at (227.3, 92.5)
- added C16: 22u, Capacitor_SMD:C_1206_3216Metric, F.Cu at (229.7, 58.6)
- added C17: 100n, Capacitor_SMD:C_0402_1005Metric, F.Cu at (233.5, 58.6)
- added C18: 22u, Capacitor_SMD:C_1206_3216Metric, F.Cu at (242.7, 58.1)
- added C19: 100n, Capacitor_SMD:C_0402_1005Metric, F.Cu at (247.1, 58.0)
- added C2: 10u, Capacitor_SMD:C_1206_3216Metric, F.Cu at (20.3, 32.1)
- added C20: 100n, Capacitor_SMD:C_0402_1005Metric, F.Cu at (222.2, 92.5)
- added C21: 100n, Capacitor_SMD:C_0402_1005Metric, F.Cu at (114.4, 48.6)
- added C22: 100n, Capacitor_SMD:C_0402_1005Metric, F.Cu at (187.8, 112.0)
- added C23: 100n, Capacitor_SMD:C_0402_1005Metric, F.Cu at (138.3, 103.7)
- added C24: 100n, Capacitor_SMD:C_0402_1005Metric, F.Cu at (59.3, 87.2)
- added C25: 100n, Capacitor_SMD:C_0402_1005Metric, F.Cu at (179.3, 46.2)
- added C26: 100n, Capacitor_SMD:C_0402_1005Metric, F.Cu at (188.2, 119.2)
- added C27: 1u, Capacitor_SMD:C_0805_2012Metric, F.Cu at (59.8, 165.0)
- added C28: 100n, Capacitor_SMD:C_0402_1005Metric, F.Cu at (54.4, 164.6)
- added C29: 100n, Capacitor_SMD:C_0402_1005Metric, F.Cu at (188.2, 129.7)
- added C3: 100n, Capacitor_SMD:C_0402_1005Metric, F.Cu at (24.9, 32.1)
- added C30: 100n, Capacitor_SMD:C_0402_1005Metric, F.Cu at (187.9, 139.8)
- added C31: 100n, Capacitor_SMD:C_0402_1005Metric, F.Cu at (188.4, 149.2)
- added C32: 100n, Capacitor_SMD:C_0402_1005Metric, F.Cu at (188.8, 158.3)
- added C33: 1n, Capacitor_SMD:C_0402_1005Metric, F.Cu at (72.7, 121.8)
- added C34: 6.8n, Capacitor_SMD:C_0402_1005Metric, F.Cu at (88.4, 126.6)
- added C35: 22u, Capacitor_SMD:C_1206_3216Metric, F.Cu at (64.0, 135.4)
- added C36: 100n,500mA, Capacitor_SMD:C_0402_1005Metric, F.Cu at (66.1, 122.8)
- added C37: 22u,500mA, Capacitor_SMD:C_1206_3216Metric, F.Cu at (64.2, 128.0)
- added C38: 10p, Capacitor_SMD:C_0402_1005Metric, F.Cu at (83.5, 121.2)
- added C39: 1u, Capacitor_SMD:C_0805_2012Metric, F.Cu at (82.8, 133.1)
- added C4: 100n, Capacitor_SMD:C_0402_1005Metric, F.Cu at (28.5, 32.0)
- added C40: 22u, Capacitor_SMD:C_1206_3216Metric, F.Cu at (59.2, 122.0)
- added C5: 100n, Capacitor_SMD:C_0402_1005Metric, F.Cu at (32.1, 32.0)
- added C6: 100n, Capacitor_SMD:C_0402_1005Metric, F.Cu at (36.4, 31.9)
- added C7: 100n, Capacitor_SMD:C_0402_1005Metric, F.Cu at (41.2, 32.1)
- added C8: 100n, Capacitor_SMD:C_0402_1005Metric, F.Cu at (45.3, 32.2)
- added C9: 1u, Capacitor_SMD:C_0805_2012Metric, F.Cu at (59.5, 32.5)
- added F1: 3A, Fuse:Fuse_1812_4532Metric, F.Cu at (-0.71, 113.5)
- added FB1: 600@100MHz, Inductor_SMD:L_1206_3216Metric, F.Cu at (52.9, 28.1)
- added FB2: 600@100MHz, Inductor_SMD:L_1206_3216Metric, F.Cu at (52.9, 35.7)
- added FB3: 600@100MHz, Inductor_SMD:L_1206_3216Metric, F.Cu at (71.5, 31.7)
- added FB5: 600@100MHz, Inductor_SMD:L_1206_3216Metric, F.Cu at (237.7, 57.7)
- added J10: DMX, Connector_JST:JST_XH_B4B-XH-A_1x04_P2.50mm_Vertical, F.Cu at (175.0, 139.2)
- added J11: DMX, Connector_JST:JST_XH_B4B-XH-A_1x04_P2.50mm_Vertical, F.Cu at (175.5, 148.8)
- added J12: DMX, Connector_JST:JST_XH_B4B-XH-A_1x04_P2.50mm_Vertical, F.Cu at (175.3, 159.1)
- added J13: USB_B, SamacSys:USBBSRA, B.Cu at (-14.8, 118.6)
- added J3: BTN, Connector_IDC:IDC-Header_2x03_P2.54mm_Vertical, F.Cu at (125.6, 101.3)
- added J4: BTN, Connector_IDC:IDC-Header_2x03_P2.54mm_Vertical, F.Cu at (126.0, 119.1)
- added J5: BTN, Connector_IDC:IDC-Header_2x03_P2.54mm_Vertical, F.Cu at (126.3, 138.2)
- added J6: BTN, Connector_IDC:IDC-Header_2x03_P2.54mm_Vertical, F.Cu at (125.3, 156.1)
- added J7: DMX, Connector_JST:JST_XH_B4B-XH-A_1x04_P2.50mm_Vertical, F.Cu at (175.5, 111.6)
- added J8: DMX, Connector_JST:JST_XH_B4B-XH-A_1x04_P2.50mm_Vertical, F.Cu at (175.7, 119.7)
- added J9: DMX, Connector_JST:JST_XH_B4B-XH-A_1x04_P2.50mm_Vertical, F.Cu at (175.2, 129.7)
- added L1: 470n, Inductor_SMD:L_0805_2012Metric, F.Cu at (72.0, 134.1)
- added R1: 10k, Resistor_SMD:R_0603_1608Metric, F.Cu at (32.8, 52.0)
- added R10: 1k, Resistor_SMD:R_0805_2012Metric, F.Cu at (258.6, 75.3)
- added R11: 4.7k, Resistor_SMD:R_0805_2012Metric, F.Cu at (258.6, 80.4)
- added R12: 1k, Resistor_SMD:R_0805_2012Metric, F.Cu at (237.4, 79.0)
- added R13: 1k, Resistor_SMD:R_0805_2012Metric, F.Cu at (242.5, 79.0)
- added R14: 4.7k, Resistor_SMD:R_0805_2012Metric, F.Cu at (247.5, 79.0)
- added R15: 1k, Resistor_SMD:R_0805_2012Metric, F.Cu at (267.4, 75.0)
- added R16: 1k, Resistor_SMD:R_0805_2012Metric, F.Cu at (267.4, 80.0)
- added R17: 4.7k, Resistor_SMD:R_0805_2012Metric, F.Cu at (267.4, 69.9)
- added R18: 4.7k, Resistor_SMD:R_0805_2012Metric, F.Cu at (267.4, 64.8)
- added R19: 100k, Resistor_SMD:R_0805_2012Metric, F.Cu at (120.3, 46.7)
- added R2: 1k, Resistor_SMD:R_0805_2012Metric, F.Cu at (226.2, 69.7)
- added R20: 100k, Resistor_SMD:R_0805_2012Metric, F.Cu at (126.9, 57.9)
- added R21: 100k, Resistor_SMD:R_0805_2012Metric, F.Cu at (64.4, 49.6)
- added R22: 20, Resistor_SMD:R_0805_2012Metric, F.Cu at (77.4, 133.4)
- added R23: 40.2k, Resistor_SMD:R_0805_2012Metric, F.Cu at (78.1, 127.3)
- added R24: 4.7k, Resistor_SMD:R_0805_2012Metric, F.Cu at (174.3, 55.5)
- added R25: 4.7k, Resistor_SMD:R_0805_2012Metric, F.Cu at (166.7, 55.5)
- added R26: 13k, Resistor_SMD:R_0805_2012Metric, F.Cu at (78.4, 121.5)
- added R27: 100k, Resistor_SMD:R_0805_2012Metric, F.Cu at (89.2, 133.3)
- added R28: 40.2k, Resistor_SMD:R_0805_2012Metric, F.Cu at (83.0, 126.7)
- added R3: 4.49k, Resistor_SMD:R_0805_2012Metric, F.Cu at (221.1, 69.5)
- added R4: 1k, Resistor_SMD:R_0805_2012Metric, F.Cu at (232.3, 79.0)
- added R5: 220, Resistor_SMD:R_0805_2012Metric, F.Cu at (258.9, 95.1)
- added R6: 220, Resistor_SMD:R_0805_2012Metric, F.Cu at (264.9, 94.2)
- added R7: 4.7k, Resistor_SMD:R_0805_2012Metric, F.Cu at (266.8, 48.3)
- added R8: 4.7k, Resistor_SMD:R_0805_2012Metric, F.Cu at (258.6, 65.1)
- added R9: 1k, Resistor_SMD:R_0805_2012Metric, F.Cu at (258.6, 70.2)
- R29, R30, R31, R32: footprint Resistor_SMD:R_0402_1005Metric -> Resistor_SMD:R_0805_2012Metric
- moved H4 594.3 mm to (5.95, 5.35)
- moved H1 574.2 mm to (16.4, 5.50)
- moved H6 557.9 mm to (2.55, 201.2)
- moved H3 533.8 mm to (10.4, 201.6)
- moved H5 369.5 mm to (290.0, 4.20)
- moved H2 353.8 mm to (279.8, 4.15)
- moved J1 297.6 mm to (237.4, 89.9)
- moved IC3 285.3 mm to (56.6, 168.2)
- moved D1 284.7 mm to (261.8, 46.3)
- moved H7 282.7 mm to (290.3, 203.5)
- moved R32 228.7 mm to (101.4, 190.9)
- moved R31 228.7 mm to (100.7, 185.2)
- moved R30 227.9 mm to (100.4, 180.7)
- moved R29 227.9 mm to (99.3, 176.5)
- moved J14 218.4 mm to (91.8, 183.7)
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
Commit message: fix usb conn
Parts:
- removed J13: USB_B, SamacSys:USBBSRA
- added J15: USB-B-S-RA, SamacSys:USBBSRA, B.Cu at (-42.5, 87.0)
- C1, C10, C2, C3, C4, C5, C6, C7, C8, C9: moved to B.Cu
- moved C1 107.6 mm to (-10.8, 93.7), turned to 180 degrees
- moved C9 93.6 mm to (-12.8, 92.0), turned to 180 degrees
- moved C10 93.5 mm to (-7.67, 92.8)
- moved R1 90.3 mm to (-34.6, 112.0), turned to 180 degrees
- moved R21 89.4 mm to (-18.3, 83.4)
- moved SW1 88.1 mm to (-39.6, 111.3), turned to -90 degrees
- moved C4 87.9 mm to (-23.0, 103.3), turned to 180 degrees
- moved C6 86.2 mm to (-9.35, 105.0), turned to -90 degrees
- moved C8 84.7 mm to (-7.67, 98.3)
- moved FB3 81.4 mm to (6.63, 80.9), turned to -135 degrees
- moved C7 79.0 mm to (-7.67, 94.3)
- moved FB1 75.1 mm to (3.16, 84.3), turned to -135 degrees
- moved C3 73.8 mm to (-21.4, 89.6), turned to 90 degrees
- moved C2 73.5 mm to (-15.3, 96.5)
- moved U1 72.9 mm to (-15.3, 97.3), turned to 180 degrees
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Connections:
- net MP2331H_SW_AFTERIND renamed +3.3V
- IC4 pad 3: MP2331H_SW -> Net-(IC4-SW)
- L1 pad 1: MP2331H_SW -> Net-(IC4-SW)
- U1 pad 70: unconnected-(U1-PA11-Pad70) -> STM_USB_D-
- U1 pad 71: unconnected-(U1-PA12-Pad71) -> STM_USB_D+

Commit message: start placing pcb
Parts:
- removed FB1, FB2, FB3: 600@100MHz, Inductor_SMD:L_1206_3216Metric
- removed R20: 100k, Resistor_SMD:R_0805_2012Metric
- C1, C10, C3, C4, C5, C6, C7, C8: moved to F.Cu
- D1, J1, J10, J11, J12, J14, J2, J3, J4, J5, J6, J7, J8, J9, R1, SW1: moved to B.Cu
- moved R6 232.9 mm to (32.9, 115.4), turned to 180 degrees
- moved R5 224.6 mm to (34.3, 97.0), turned to 180 degrees
- moved C14 219.7 mm to (51.3, 96.3), turned to 180 degrees
- moved R7 216.7 mm to (55.5, 96.3), turned to 180 degrees
- moved D1 212.0 mm to (53.6, 86.4)
- moved R18 204.7 mm to (65.4, 98.0), turned to 180 degrees
- moved R17 203.6 mm to (66.0, 100.1), turned to 180 degrees
- moved R15 202.4 mm to (66.8, 102.2), turned to 180 degrees
- moved R16 201.2 mm to (67.6, 104.3), turned to 180 degrees
- moved R8 200.7 mm to (66.3, 122.5), turned to 180 degrees
- moved R9 198.4 mm to (66.7, 120.4), turned to 180 degrees
- moved C19 197.7 mm to (55.5, 106.9), turned to 180 degrees
- moved C18 196.8 mm to (52.0, 106.6), turned to 180 degrees
- moved R10 195.9 mm to (67.5, 118.3), turned to 180 degrees
- moved J1 195.5 mm to (43.0, 110.9), turned to 90 degrees
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Connections:
- C1 pad 1: +3.3VREF -> +3.3V
- C1 pad 2: GNDA -> GND
- C10 pad 1: +3.3VA -> +3.3V
- C10 pad 2: GNDA -> GND
- C12 pad 1: KSZ_VDD_1.2V -> KSZ_VDD_1.2
- C13 pad 1: KSZ_VDD_1.2V -> KSZ_VDD_1.2
- C9 pad 1: +3.3VA -> +3.3V
- C9 pad 2: GNDA -> GND
- IC4 pad 3: Net-(IC4-SW) -> MP2331H_SW
- L1 pad 1: Net-(IC4-SW) -> MP2331H_SW
- U1 pad 20: GNDA -> GND
- U1 pad 21: +3.3VREF -> +3.3V
- U1 pad 22: +3.3VA -> +3.3V

Commit message: fill buy links
Parts:
- C14: value 10u -> pol_10u; footprint Capacitor_SMD:C_1206_3216Metric -> Capacitor_SMD:C_0603_1608Metric
- C2, C9, R1: moved to F.Cu
- D1: value 1N4148 -> 1N4148WT; footprint Diode_THT:D_DO-35_SOD27_P7.62mm_Horizontal -> Diode_SMD:D_SOD-523; moved to F.Cu
- J3, J4, J5, J6: footprint Connector_IDC:IDC-Header_2x03_P2.54mm_Vertical -> Connector_JST:JST_XH_B6B-XH-A_1x06_P2.50mm_Vertical
- R10, R11, R12, R13, R14, R15, R16, R17, R18, R19, R2, R21, R24, R25, R27, R4, R7, R8, R9: footprint Resistor_SMD:R_0805_2012Metric -> Resistor_SMD:R_0603_1608Metric
- R3: value 4.49k -> 6.49k
- moved J5 16.0 mm to (72.5, 48.9), turned to 0 degrees
- moved C9 15.8 mm to (45.6, 64.5)
- moved J6 13.7 mm to (91.6, 49.0), turned to 0 degrees
- moved C2 12.4 mm to (65.3, 47.5), turned to 0 degrees
- moved D1 8.06 mm to (55.2, 94.2), turned to 180 degrees
- moved J4 5.42 mm to (84.0, 30.4), turned to 180 degrees
- moved J3 3.34 mm to (102.8, 30.5), turned to 180 degrees
