File: kp_artnet2dmx6.kicad_pcb (KiCad board)
At the start: 4 copper layers, 95 x 104 mm, 99 parts, among them IC1 KSZ8081MNXIA-TR, IC2 M95640-RMN6P, IC3 AP2281-3WG-7, IC4 MP2331HGTL-P, J1 RJ45_Amphenol_RJMG1BD3B8K1ANR, J10 DMX, J11 DMX, J12 DMX, J14 SWD, J15 USB-B-S-RA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

Commit message: DRC OK
Parts:
- L1: footprint Inductor_SMD:L_0805_2012Metric -> homemade_footprints:L_Bourns_SRP4020CC
- moved C34 15.1 mm to (75.5, 47.6), turned to 0 degrees
- moved C38 14.5 mm to (70.8, 52.1)
- moved R22 12.7 mm to (78.0, 52.2), turned to -90 degrees
- moved R28 12.6 mm to (72.4, 52.2), turned to -90 degrees
- moved C39 12.3 mm to (80.0, 52.2), turned to 90 degrees
- moved R27 11.4 mm to (75.9, 46.2)
- moved R26 10.5 mm to (73.8, 49.4), turned to 0 degrees
- moved R23 10.3 mm to (74.5, 52.2)
- moved C35 9.92 mm to (82.0, 63.0), turned to 180 degrees
- moved L1 9.27 mm to (81.5, 56.5), turned to 0 degrees
- moved C40 8.37 mm to (81.9, 60.4), turned to 180 degrees
- moved IC4 6.39 mm to (76.3, 56.1)
- moved C33 5.89 mm to (73.0, 58.5)
- moved C28 5.81 mm to (67.7, 42.7)
- moved IC3 5.81 mm to (67.3, 45.7)
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Routing:
- net Earth: track 19.2 -> 51.0 mm, vias 5 -> 8
- net GND: track 122.7 -> 109.3 mm, vias 40 -> 38
- net STM_PWR_5V_EN_GPIO: track 65.3 -> 75.2 mm
- net +3.3V: track 120.4 -> 112.3 mm
- net /mp2331_ss: track 1.12 -> 7.84 mm
- net /mp2331_fb2: track 0.00 -> 5.85 mm
- net +5V_IN: track 27.2 -> 31.5 mm
- net /mp2331_en: track 5.04 -> 9.26 mm
- net /mp2331_fb1: track 0.00 -> 2.76 mm
- net KSZ_LED0: track 44.2 -> 46.7 mm
- net /ksz_led0+: track 5.16 -> 3.96 mm
- net /mp2331_pg: track 2.01 -> 3.14 mm
- net /mp2331_bst1: track 1.68 -> 2.73 mm
- net /mp2331_bst2: track 2.63 -> 2.02 mm

Commit message: add pwr leds
Parts:
- added D2: LED, LED_SMD:LED_0805_2012Metric, F.Cu at (61.0, 46.1)
- added D3: LED, LED_SMD:LED_0805_2012Metric, F.Cu at (70.5, 64.0)
- added D4: LED, LED_SMD:LED_0805_2012Metric, F.Cu at (123.5, 117.9)
- added D5: LED, LED_SMD:LED_0805_2012Metric, F.Cu at (132.9, 43.4)
- added R20: 3k, Resistor_SMD:R_0805_2012Metric, F.Cu at (58.4, 43.5)
- added R33: 3k, Resistor_SMD:R_0805_2012Metric, F.Cu at (73.1, 66.6)
- added R34: 1k, Resistor_SMD:R_0603_1608Metric, F.Cu at (121.0, 115.4)
- added R35: 3k, Resistor_SMD:R_0805_2012Metric, F.Cu at (130.4, 40.9)
Routing:
- net +5V: track 12.5 -> 18.1 mm, vias 5 -> 6
- net +5V_USB: track 13.7 -> 19.2 mm
- net +5V_IN: track 31.5 -> 34.6 mm
- net +3.3V: track 112.3 -> 114.7 mm, vias 24 -> 25
- net /led1: track 0.00 -> 1.85 mm
- net /led2: track 0.00 -> 1.80 mm
- net /led3: track 0.00 -> 1.77 mm
- net /led4: track 0.00 -> 1.77 mm
Other:
- board text added: "PWR3.3"
- board text added: "PWR5"
- board text added: "PWRIN"
- board text added: "PWRUSB"
