File: kp_artnet2dmx6.kicad_sch (KiCad schematic)
At the start: 112 parts, among them IC1 KSZ8081MNXIA-TR, IC2 M95640-RMN6P, IC3 AP2281-3WG-7, IC4 MP2331HGTL-P, J1 RJ45_Amphenol_RJMG1BD3B8K1ANR, J10 DMX, J11 DMX, J12 DMX, J14 SWD, J15 USB-B-S-RA, J2 SCREEN, J3 BTN, J4 BTN, J5 BTN, J6 BTN, J7 DMX, J8 DMX, J9 DMX, Q1 AO3401A, SW1 SW_SPDT, U1 STM32F407VETx, U2 MCP23S17_SP, U3 USBLC6-2SC6, Y1 ASDDV-25.000MHZ-LC-T

Commit message: start placing pcb
Parts:
- removed FB1, FB2, FB3: 600@100MHz, Inductor_SMD:L_1206_3216Metric, symbol Device:FerriteBead_Small
- removed R20: 100k, Resistor_SMD:R_0805_2012Metric, symbol Device:R_Small
- J15: footprint USBBSRA -> SamacSys:USBBSRA
Connections:
- net +3.3VA is gone; now on net +3.3V: C10.1, C9.1, U1.22 (VDDA)
- net +3.3VREF is gone; now on net +3.3V: C1.1, U1.21 (VREF+)
- net GNDA is gone; now on net GND: C1.2, C10.2, C9.2, U1.20 (VSSA)
- net KSZ_VDD_1.2V is gone; now on net KSZ_VDD_1.2: C12.1, C13.1
- net MP2331H_SW: now also IC4.3 (SW), L1.1
Other:
- note added: "VDDA"
- note added: "VREF"
- note added: "for eeprom, cf datasheet p.6"
- note removed: "for eeprom, cf datasheet p.11"

Commit message: fill buy links
Parts:
- removed D1: 1N4148, Diode_THT:D_DO-35_SOD27_P7.62mm_Horizontal, symbol Diode:1N4148
- added D1: 1N4148WT, Diode_SMD:D_SOD-523, symbol Diode:1N4148WT
- C1, C10, C13, C15, C17, C19, C20, C21, C22, C23, C24, C25, C26, C28, C29, C3, C30, C31, C32, C36, C4, C5, C6, C7, C8: JLCPCB Part # (none) -> C1525
- C11: JLCPCB Part # (none) -> C15195
- C12: JLCPCB Part # (none) -> C19110
- C14: value 10u -> pol_10u; footprint Capacitor_SMD:C_1206_3216Metric -> Capacitor_SMD:C_0603_1608Metric; JLCPCB Part # (none) -> C2158420
- C2: JLCPCB Part # (none) -> C9807
- C27, C39, C9: JLCPCB Part # (none) -> C24123
- C33: JLCPCB Part # (none) -> C14442
- C34: JLCPCB Part # (none) -> C161171
- C38: JLCPCB Part # (none) -> C32949
- IC3: JLCPCB Part # (none) -> C128634
- IC4: farnell link (none) -> https://fr.farnell.com/monolithic-power-systems-mps/mp2331h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
- J10, J11, J12, J2, J7, J8, J9: farnell link (none) -> https://www.lcsc.com/product-detail/C144395.html?s_z=n_B4B-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
- J14: farnell link (none) -> https://www.lcsc.com/product-detail/C46061719.html
- J3, J4, J5, J6: footprint Connector_IDC:IDC-Header_2x03_P2.54mm_Vertical -> Connector_JST:JST_XH_B6B-XH-A_1x06_P2.50mm_Vertical; farnell link (none) -> https://www.lcsc.com/product-detail/C144397.html?s_z=n_B6B-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
- Q1: JLCPCB Part # (none) -> C15127
- R1: JLCPCB Part # (none) -> C844918
- R10, R12, R13, R15, R16, R2, R4, R9: footprint Resistor_SMD:R_0805_2012Metric -> Resistor_SMD:R_0603_1608Metric; JLCPCB Part # (none) -> C844920
- R11, R14, R17, R18, R24, R25, R7, R8: footprint Resistor_SMD:R_0805_2012Metric -> Resistor_SMD:R_0603_1608Metric; JLCPCB Part # (none) -> C23162
- R19, R21, R27: footprint Resistor_SMD:R_0805_2012Metric -> Resistor_SMD:R_0603_1608Metric; JLCPCB Part # (none) -> C2907088
- R22: JLCPCB Part # (none) -> C17544
- R23, R28: JLCPCB Part # (none) -> C17678
- R26: JLCPCB Part # (none) -> C17455
- R29, R30, R31, R32: JLCPCB Part # (none) -> C17561
- R3: value 4.49k -> 6.49k; JLCPCB Part # (none) -> C2933484
- R5, R6: JLCPCB Part # (none) -> C2933537
- SW1: farnell link (none) -> https://fr.farnell.com/c-k-components/pcm12smtr/commutateur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
- TP1: now left out of the parts list
- U1: value STM32F407VETx -> STM32F407VGT6; JLCPCB Part # (none) -> C12345
- U2: farnell link (none) -> already have
- U3: JLCPCB Part # (none) -> C7519
- Y1: JLCPCB Part # (none) -> C1857781
Connections:
- net +3.3V: now also D1.1 (K)
- net KSZ_RST: now also D1.2 (A)
