File: kp_dmxinout/kp_dmxinout.kicad_sch (KiCad schematic)
At the start: 25 parts, among them J1 NC3MAAH, J2 NC3FAAH, J3 Conn_01x04, U1 SN75176AD, U2 6N137, U3 6N137, U4 SN75176AD

Commit message: invert dmx out DATA+ & DATA-
Connections:
- net IN_DATA+: now also J1.3; no longer J1.2
- net IN_DATA-: now also J1.2; no longer J1.3
- net OUT_DATA+: now also J2.3; no longer J2.2
- net OUT_DATA-: now also J2.2; no longer J2.3
